File: electronique/electronique.kicad_pcb (KiCad board)
At the start: 2 copper layers, 70 x 50 mm, 47 parts, among them J1 Conn_01x02, J10 PHOTOD3, J11 PHOTOD4, J12 Ultrason 3, J13 Moteur 1, J14 Moteur 2, J2 Conn_02x07_Odd_Even, J3 Camera, J4 TOF1, J5 Conn_01x06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

Commit message: Example commit sur autre branche
Routing:
- net /PHOTOD_COUL: track 0.00 -> 40.9 mm, vias 0 -> 1
- net /LED_A: track 0.00 -> 38.7 mm, vias 0 -> 1
- net /LED_B: track 0.00 -> 36.9 mm, vias 0 -> 1
- net /LED_C: track 0.00 -> 34.4 mm, vias 0 -> 1

Commit message: Circuit routé attente de validation
Parts:
- moved C3 1.75 mm to (46.2, 43.0)
- moved C6 1.75 mm to (46.2, 45.2)
- moved C1 1.60 mm to (46.2, 25.0)
- moved C4 1.35 mm to (56.5, 42.0), turned to 270 degrees
- moved C7 1.03 mm to (39.5, 38.0)
- moved C8 1.00 mm to (41.8, 38.0)
- moved U3 0.75 mm to (37.2, 57.0)
Routing:
- net /M2_A: track 0.00 -> 59.6 mm, vias 0 -> 3
- net /M2_B: track 0.50 -> 58.6 mm, vias 0 -> 3
- net GND: track 63.8 -> 115.0 mm, vias 7 -> 18
- net /M1_PWM: track 0.00 -> 40.5 mm, vias 0 -> 2
- net +3V3: track 198.7 -> 239.0 mm, vias 0 -> 2
- net /SWDIO: track 0.00 -> 39.0 mm, vias 0 -> 2
- net /I_SENS1: track 0.00 -> 38.9 mm, vias 0 -> 2
- net /M1N_PWM: track 0.00 -> 38.3 mm, vias 0 -> 4
- net +5V: track 82.2 -> 119.5 mm, vias 1 -> 3
- net /M1_B: track 0.00 -> 36.1 mm, vias 0 -> 1
- net /I_SENS2: track 0.00 -> 32.8 mm, vias 0 -> 2
- net /RX1: track 0.00 -> 32.8 mm
- net /SWCLK: track 0.00 -> 32.4 mm, vias 0 -> 2
- net /SCL: track 0.00 -> 32.3 mm
- net /M1_A: track 0.00 -> 32.2 mm, vias 0 -> 1
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